Commit message: extender_arduino package works

File: src/minibot/description/ros2_control.xacro (robot description, xacro)
@@ -22,4 +22,23 @@
             </joint>
             <joint name="right_wheel_joint">
+                <command_interface name="velocity">
+                    <param name="min">-10</param>
+                    <param name="max">10</param>
+                </command_interface>
+                <state_interface name="position"/>
+                <state_interface name="velocity"/>
+            </joint>
+        </ros2_control>
+        <ros2_control name="GrabberSystem" type="system">
+            <hardware>
+                <plugin>extender_arduino/ExtenderArduinoHardware</plugin>
+                    <param name="joints">slider_left_joint</param>
+                    <param name="loop_rate">30</param>
+                    <param name="device">/dev/ttyACM1</param>
+                    <param name="baud_rate">57600</param>
+                    <param name="timeout_ms">1000</param>
+                    <param name="enc_counts_per_rev">3200</param>
+            </hardware>
+            <joint name="slider_left_joint">
                 <command_interface name="velocity">
                     <param name="min">-10</param>
