Commit message: Update robot_main.xacro

File: src/minibot/description/robot_main.xacro (robot description, xacro)
@@ -2,13 +2,13 @@
 <robot xmlns:xacro="http://www.ros.org/wiki/xacro">
     <xacro:include filename = "inertial_macros.xacro" />
-    <xacro:property name="chassis_length"           value="0.320"/>
-    <xacro:property name="chassis_width"            value="0.240"/>
-    <xacro:property name="chassis_height"           value="0.078"/>
+    <xacro:property name="chassis_length"           value="0.464"/>
+    <xacro:property name="chassis_width"            value="0.48"/>
+    <xacro:property name="chassis_height"           value="0.3"/>
     <xacro:property name="chassis_mass"             value="0.700"/>
-    <xacro:property name="wheel_radius"             value="0.034"/>
-    <xacro:property name="wheel_thickness"          value="0.026"/>
+    <xacro:property name="wheel_radius"             value="0.1"/>
+    <xacro:property name="wheel_thickness"          value="0.08"/>
     <xacro:property name="wheel_mass"               value="0.050"/>
     <xacro:property name="wheel_offset_x"           value="0.133"/>
-    <xacro:property name="wheel_offset_y"           value="0.133"/>
+    <xacro:property name="wheel_offset_y"           value="0.275"/>
     <xacro:property name="wheel_offset_z"           value="0.020"/>
     <xacro:property name="caster_wheel_radius"      value="${wheel_radius - wheel_offset_z}"/>
@@ -32,4 +32,7 @@
         <color rgba= "0.294 0 0.51 1"/>
     </material>
+    <material name="blue">
+        <color rgba= "0 0 1 1"/>
+    </material>
     <!-- convention (except base_link): joint followed by link -->
     <!-- base_link -->
@@ -150,3 +153,103 @@
         <mu2 value= "0.0001"/>
     </gazebo>
+    <!--Extender Left Arm-->
+    <joint name="extender_left_arm_joint" type="fixed">
+        <parent link= "chasis"/>
+        <child link= "extender_left_arm"/>
+        <origin xyz= "${chassis_length+0.15} 0.1 ${wheel_offset_z}" rpy= "0 0 0"/>
+    </joint>
+    <link name="extender_left_arm">
+        <visual>
+            <origin xyz= "0 0 0" rpy= "0 0 0"/>
+            <geometry>
+                <box size = "0.3 0.05 0.05"/>
+            </geometry>
+            <material name= "blue"/>
+        </visual>
+        <collision>
+            <origin xyz= "0 0 0" rpy= "0 0 0"/>
+            <geometry>
+                <box size = "0.3 0.05 0.05"/>
+            </geometry>
+        </collision>
+        <xacro:inertial_box mass= "0.5" x="0.1" y="0.1" z="0.1">
+            <origin xyz= "0 0 0" rpy= "0 0 0"/>
+        </xacro:inertial_box>
+    </link>
+    <!--Extender Right Arm-->
+    <joint name="extender_right_arm_joint" type="fixed">
+        <parent link= "chasis"/>
+        <child link= "extender_right_arm"/>
+        <origin xyz= "${chassis_length+0.15} -0.1 ${wheel_offset_z}" rpy= "0 0 0"/>
+    </joint>
+    <link name="extender_right_arm">
+        <visual>
+            <origin xyz= "0 0 0" rpy= "0 0 0"/>
+            <geometry>
+                <box size = "0.3 0.05 0.05"/>
+            </geometry>
+            <material name= "blue"/>
+        </visual>
+        <collision>
+            <origin xyz= "0 0 0" rpy= "0 0 0"/>
+            <geometry>
+                <box size = "0.3 0.05 0.05"/>
+            </geometry>
+        </collision>
+        <xacro:inertial_box mass= "0.5" x="0.1" y="0.1" z="0.1">
+            <origin xyz= "0 0 0" rpy= "0 0 0"/>
+        </xacro:inertial_box>
+    </link>
+    <!-- Slider on Extender Left Arm -->
+    <joint name="slider_left_joint" type="prismatic">
+        <parent link="extender_left_arm"/>
+        <child link="slider_left"/>
+        <origin xyz="0 0 0" rpy="0 0 0"/>
+        <axis xyz="1 0 0"/>
+        <limit lower="0" upper="0.3" effort="10" velocity="0.1"/>
+    </joint>
+    <link name="slider_left">
+        <visual>
+            <origin xyz="0.05 0 0.025" rpy="0 0 0"/>
+            <geometry>
+                <box size="0.3 0.05 0.01"/>
+            </geometry>
+            <material name="white"/>
+        </visual>
+        <collision>
+            <origin xyz="0.05 0 0.025" rpy="0 0 0"/>
+            <geometry>
+                <box size="0.3 0.05 0.01"/>
+            </geometry>
+        </collision>
+        <xacro:inertial_box mass="0.1" x="0.3" y="0.05" z="0.01">
+            <origin xyz="0.05 0 0.025" rpy="0 0 0"/>
+        </xacro:inertial_box>
+    </link>
+    <!-- Slider on Extender Right Arm -->
+    <joint name="slider_right_joint" type="prismatic">
+        <parent link="extender_right_arm"/>
+        <child link="slider_right"/>
+        <origin xyz="0 0 0" rpy="0 0 0"/>
+        <axis xyz="1 0 0"/>
+        <limit lower="0" upper="0.3" effort="10" velocity="0.1"/>
+    </joint>
+    <link name="slider_right">
+        <visual>
+            <origin xyz="0.05 0 0.025" rpy="0 0 0"/>
+            <geometry>
+                <box size="0.3 0.05 0.01"/>
+            </geometry>
+            <material name="white"/>
+        </visual>
+        <collision>
+            <origin xyz="0.05 0 0.025" rpy="0 0 0"/>
+            <geometry>
+                <box size="0.3 0.05 0.01"/>
+            </geometry>
+        </collision>
+        <xacro:inertial_box mass="0.1" x="0.3" y="0.05" z="0.01">
+            <origin xyz="0.05 0 0.025" rpy="0 0 0"/>
+        </xacro:inertial_box>
+    </link>
 </robot>

Commit message: finished designing joint for the platform and the grippers

File: src/minibot/description/robot_main.xacro (robot description, xacro)
@@ -153,9 +153,35 @@
         <mu2 value= "0.0001"/>
     </gazebo>
+    <!--Platform-->
+    <joint name="platform_joint" type="prismatic">
+        <parent link= "chasis"/>
+        <child link= "platform"/>
+        <origin xyz= "${chassis_length+0.15} 0 ${wheel_offset_z}" rpy= "0 0 0"/>
+        <axis xyz= "0 0 1"/>
+        <limit lower="0" upper="1" effort="10" velocity="0.1"/>
+    </joint>
+    <link name="platform">
+        <visual>
+            <origin xyz= "0 0 0" rpy= "0 0 0"/>
+            <geometry>
+                <box size = "0.3 0.3 0.05"/>
+            </geometry>
+            <material name= "blue"/>
+        </visual>
+        <collision>
+            <origin xyz= "0 0 0" rpy= "0 0 0"/>
+            <geometry>
+                <box size = "0.3 0.3 0.05"/>
+            </geometry>
+        </collision>
+        <xacro:inertial_box mass= "0.5" x="0.1" y="0.1" z="0.1">
+            <origin xyz= "0 0 0" rpy= "0 0 0"/>
+        </xacro:inertial_box>
+    </link>
     <!--Extender Left Arm-->
     <joint name="extender_left_arm_joint" type="fixed">
-        <parent link= "chasis"/>
+        <parent link= "platform"/>
         <child link= "extender_left_arm"/>
-        <origin xyz= "${chassis_length+0.15} 0.1 ${wheel_offset_z}" rpy= "0 0 0"/>
+        <origin xyz= "0 0.15 ${wheel_offset_z+0.02}" rpy= "0 0 0"/>
     </joint>
     <link name="extender_left_arm">
@@ -179,7 +205,7 @@
     <!--Extender Right Arm-->
     <joint name="extender_right_arm_joint" type="fixed">
-        <parent link= "chasis"/>
+        <parent link= "platform"/>
         <child link= "extender_right_arm"/>
-        <origin xyz= "${chassis_length+0.15} -0.1 ${wheel_offset_z}" rpy= "0 0 0"/>
+        <origin xyz= "0 -0.15 ${wheel_offset_z+0.02}" rpy= "0 0 0"/>
     </joint>
     <link name="extender_right_arm">
@@ -207,5 +233,5 @@
         <origin xyz="0 0 0" rpy="0 0 0"/>
         <axis xyz="1 0 0"/>
-        <limit lower="0" upper="0.3" effort="10" velocity="0.1"/>
+        <limit lower="0" upper="0.235" effort="10" velocity="0.1"/>
     </joint>
     <link name="slider_left">
@@ -233,5 +259,5 @@
         <origin xyz="0 0 0" rpy="0 0 0"/>
         <axis xyz="1 0 0"/>
-        <limit lower="0" upper="0.3" effort="10" velocity="0.1"/>
+        <limit lower="0" upper="0.235" effort="10" velocity="0.1"/>
     </joint>
     <link name="slider_right">
@@ -253,3 +279,55 @@
         </xacro:inertial_box>
     </link>
+    <!-- gripper_left -->
+    <joint name="gripper_left_joint" type="revolute">
+        <parent link="slider_left"/>
+        <child link= "gripper_left"/>
+        <origin xyz= "0.2 0 0" rpy= "0 0 0"/>
+        <axis xyz= "0 0 1"/>
+        <limit lower="-1.57" upper="0" effort="10" velocity="0.1"/>
+    </joint>
+    <link name="gripper_left">
+        <visual>
+            <origin xyz= "0.02 0 0.0423" rpy= "0 0 0"/>
+            <geometry>
+                <box size = "0.1 0.025 0.025"/>
+            </geometry>
+            <material name= "cyan"/>
+        </visual>
+        <collision>
+            <origin xyz= "0.02 0 0.0423" rpy= "0 0 0"/>
+            <geometry>
+                <box size = "0.1 0.025 0.025"/>
+            </geometry>
+        </collision>
+        <xacro:inertial_box mass= "0.5" x="0.1" y="0.1" z="0.1">
+            <origin xyz= "0.02 0 0.0423" rpy= "0 0 0"/>
+        </xacro:inertial_box>
+    </link>
+    <!-- gripper_right -->
+    <joint name="gripper_right_joint" type="revolute">
+        <parent link="slider_right"/>
+        <child link= "gripper_right"/>
+        <origin xyz= "0.2 0 0" rpy= "0 0 0"/>
+        <axis xyz= "0 0 1"/>
+        <limit lower="0" upper="1.57" effort="10" velocity="0.1"/>
+    </joint>
+    <link name="gripper_right">
+        <visual>
+            <origin xyz= "0.02 0 0.0423" rpy= "0 0 0"/>
+            <geometry>
+                <box size = "0.1 0.025 0.025"/>
+            </geometry>
+            <material name= "cyan"/>
+        </visual>
+        <collision>
+            <origin xyz= "0.02 0 0.0423" rpy= "0 0 0"/>
+            <geometry>
+                <box size = "0.1 0.025 0.025"/>
+            </geometry>
+        </collision>
+        <xacro:inertial_box mass= "0.5" x="0.1" y="0.1" z="0.1">
+            <origin xyz= "0.02 0 0.0423" rpy= "0 0 0"/>
+        </xacro:inertial_box>
+    </link>
 </robot>
