Commit message: changes made to obtain orientation state_interface in ros2_control. Still need revise code

File: src/diffdrive_arduino/description/ros2_control/diffbot.ros2_control.xacro (robot description, xacro)
@@ -27,4 +27,9 @@
         <state_interface name="velocity"/>
       </joint>
+      <sensor name="imu_sensor">
+        <state_interface name="orientation"/>
+        <state_interface name="angular_velocity"/>
+        <state_interface name="linear_acceleration"/>
+      </sensor>
     </ros2_control>
   </xacro:macro>

File: src/diffdrive_arduino/description/urdf/diffbot_description.urdf.xacro (robot description, xacro)
@@ -158,4 +158,31 @@
         </inertial>
       </link>
+    <!-- IMU Sensor Link -->
+    <link name="${prefix}imu_link">
+      <inertial>
+        <mass value="0.01"/>
+        <origin xyz="0 0 0" rpy="0 0 0"/>
+        <inertia ixx="0.0001" ixy="0.0" ixz="0.0" iyy="0.0001" iyz="0.0" izz="0.0001"/>
+      </inertial>
+      <visual>
+        <origin xyz="0 0 0" rpy="0 0 0"/>
+        <geometry>
+          <box size="0.02 0.02 0.02"/>
+        </geometry>
+        <material name="black"/>
+      </visual>
+      <collision>
+        <origin xyz="0 0 0" rpy="0 0 0"/>
+        <geometry>
+          <box size="0.02 0.02 0.02"/>
+        </geometry>
+      </collision>
+    </link>
+    <!-- IMU Sensor Joint -->
+    <joint name="${prefix}imu_joint" type="fixed">
+      <parent link="${prefix}base_link"/>
+      <child link="${prefix}imu_link"/>
+      <origin xyz="0 0 0.1" rpy="0 0 0"/>
+    </joint>
   </xacro:macro>
 </robot>

Commit message: newly updated

File: src/diffdrive_arduino/description/ros2_control/diffbot.ros2_control.xacro (robot description, xacro)
@@ -11,9 +11,9 @@
         <param name="baud_rate">57600</param>
         <param name="timeout_ms">1000</param>
-        <param name="enc_counts_per_rev">3436</param>
-        <param name="pid_p">20</param>
-        <param name="pid_d">12</param>
-        <param name="pid_i">0</param>
-        <param name="pid_o">50</param>
+        <param name="enc_counts_per_rev">3200</param>
+        <param name="pid_p">11</param>
+        <param name="pid_d">1</param>
+        <param name="pid_i">1</param>
+        <param name="pid_o">49</param>
       </hardware>
       <joint name="${prefix}left_wheel_joint">

File: src/minibot/description/lidar.xacro (robot description, xacro)
@@ -4,5 +4,6 @@
     <xacro:property name="lidar_thickness"          value="0.040"/>
     <xacro:property name="lidar_offset_x"           value="0.230"/>
-    <xacro:property name="lidar_offset_z"           value="0.098"/>
+    <!-- <xacro:property name="lidar_offset_z"           value="0.098"/> -->
+    <xacro:property name="lidar_offset_z"           value="0.34"/>
     <!-- Lidar -->
     <joint name="lidar_joint" type="fixed">

File: src/minibot/description/robot_main.xacro (robot description, xacro)
@@ -2,13 +2,13 @@
 <robot xmlns:xacro="http://www.ros.org/wiki/xacro">
     <xacro:include filename = "inertial_macros.xacro" />
-    <xacro:property name="chassis_length"           value="0.320"/>
-    <xacro:property name="chassis_width"            value="0.240"/>
-    <xacro:property name="chassis_height"           value="0.078"/>
+    <xacro:property name="chassis_length"           value="0.464"/>
+    <xacro:property name="chassis_width"            value="0.48"/>
+    <xacro:property name="chassis_height"           value="0.3"/>
     <xacro:property name="chassis_mass"             value="0.700"/>
-    <xacro:property name="wheel_radius"             value="0.034"/>
-    <xacro:property name="wheel_thickness"          value="0.026"/>
+    <xacro:property name="wheel_radius"             value="0.1"/>
+    <xacro:property name="wheel_thickness"          value="0.08"/>
     <xacro:property name="wheel_mass"               value="0.050"/>
     <xacro:property name="wheel_offset_x"           value="0.133"/>
-    <xacro:property name="wheel_offset_y"           value="0.133"/>
+    <xacro:property name="wheel_offset_y"           value="0.275"/>
     <xacro:property name="wheel_offset_z"           value="0.020"/>
     <xacro:property name="caster_wheel_radius"      value="${wheel_radius - wheel_offset_z}"/>
@@ -31,4 +31,7 @@
     <material name="indigo">
         <color rgba= "0.294 0 0.51 1"/>
+    </material>
+    <material name="blue">
+        <color rgba= "0 0 1 1"/>
     </material>
     <!-- convention (except base_link): joint followed by link -->
@@ -150,3 +153,205 @@
         <mu2 value= "0.0001"/>
     </gazebo>
+    <!--Platform-->
+    <joint name="platform_joint" type="prismatic">
+        <parent link= "chasis"/>
+        <child link= "platform"/>
+        <origin xyz= "${chassis_length+0.15} 0 ${wheel_offset_z}" rpy= "0 0 0"/>
+        <axis xyz= "0 0 1"/>
+        <limit lower="0" upper="1" effort="10" velocity="0.1"/>
+    </joint>
+    <link name="platform">
+        <visual>
+            <origin xyz= "0 0 0" rpy= "0 0 0"/>
+            <geometry>
+                <box size = "0.3 0.3 0.05"/>
+            </geometry>
+            <material name= "blue"/>
+        </visual>
+        <collision>
+            <origin xyz= "0 0 0" rpy= "0 0 0"/>
+            <geometry>
+                <box size = "0.3 0.3 0.05"/>
+            </geometry>
+        </collision>
+        <xacro:inertial_box mass= "0.5" x="0.1" y="0.1" z="0.1">
+            <origin xyz= "0 0 0" rpy= "0 0 0"/>
+        </xacro:inertial_box>
+    </link>
+    <!--Extender Left Arm-->
+    <joint name="extender_left_arm_joint" type="fixed">
+        <parent link= "platform"/>
+        <child link= "extender_left_arm"/>
+        <origin xyz= "0 0.15 ${wheel_offset_z+0.02}" rpy= "0 0 0"/>
+    </joint>
+    <link name="extender_left_arm">
+        <visual>
+            <origin xyz= "0 0 0" rpy= "0 0 0"/>
+            <geometry>
+                <box size = "0.3 0.05 0.05"/>
+            </geometry>
+            <material name= "blue"/>
+        </visual>
+        <collision>
+            <origin xyz= "0 0 0" rpy= "0 0 0"/>
+            <geometry>
+                <box size = "0.3 0.05 0.05"/>
+            </geometry>
+        </collision>
+        <xacro:inertial_box mass= "0.5" x="0.1" y="0.1" z="0.1">
+            <origin xyz= "0 0 0" rpy= "0 0 0"/>
+        </xacro:inertial_box>
+    </link>
+    <!--Extender Right Arm-->
+    <joint name="extender_right_arm_joint" type="fixed">
+        <parent link= "platform"/>
+        <child link= "extender_right_arm"/>
+        <origin xyz= "0 -0.15 ${wheel_offset_z+0.02}" rpy= "0 0 0"/>
+    </joint>
+    <link name="extender_right_arm">
+        <visual>
+            <origin xyz= "0 0 0" rpy= "0 0 0"/>
+            <geometry>
+                <box size = "0.3 0.05 0.05"/>
+            </geometry>
+            <material name= "blue"/>
+        </visual>
+        <collision>
+            <origin xyz= "0 0 0" rpy= "0 0 0"/>
+            <geometry>
+                <box size = "0.3 0.05 0.05"/>
+            </geometry>
+        </collision>
+        <xacro:inertial_box mass= "0.5" x="0.1" y="0.1" z="0.1">
+            <origin xyz= "0 0 0" rpy= "0 0 0"/>
+        </xacro:inertial_box>
+    </link>
+    <!-- Slider on Extender Left Arm -->
+    <joint name="slider_left_joint" type="prismatic">
+        <parent link="extender_left_arm"/>
+        <child link="slider_left"/>
+        <origin xyz="0 0 0" rpy="0 0 0"/>
+        <axis xyz="1 0 0"/>
+        <limit lower="0" upper="0.235" effort="10" velocity="0.1"/>
+    </joint>
+    <link name="slider_left">
+        <visual>
+            <origin xyz="0.05 0 0.025" rpy="0 0 0"/>
+            <geometry>
+                <box size="0.3 0.05 0.01"/>
+            </geometry>
+            <material name="white"/>
+        </visual>
+        <collision>
+            <origin xyz="0.05 0 0.025" rpy="0 0 0"/>
+            <geometry>
+                <box size="0.3 0.05 0.01"/>
+            </geometry>
+        </collision>
+        <xacro:inertial_box mass="0.1" x="0.3" y="0.05" z="0.01">
+            <origin xyz="0.05 0 0.025" rpy="0 0 0"/>
+        </xacro:inertial_box>
+    </link>
+    <!-- Slider on Extender Right Arm -->
+    <joint name="slider_right_joint" type="fixed">
+        <parent link="slider_left"/>
+        <child link="slider_right"/>
+        <origin xyz="0 -0.3 0" rpy="0 0 0"/>
+        <!-- <axis xyz="1 0 0"/> -->
+        <!-- <limit lower="0" upper="0.235" effort="10" velocity="0.1"/> -->
+    </joint>
+    <link name="slider_right">
+        <visual>
+            <origin xyz="0.05 0 0.025" rpy="0 0 0"/>
+            <geometry>
+                <box size="0.3 0.05 0.01"/>
+            </geometry>
+            <material name="white"/>
+        </visual>
+        <collision>
+            <origin xyz="0.05 0 0.025" rpy="0 0 0"/>
+            <geometry>
+                <box size="0.3 0.05 0.01"/>
+            </geometry>
+        </collision>
+        <xacro:inertial_box mass="0.1" x="0.3" y="0.05" z="0.01">
+            <origin xyz="0.05 0 0.025" rpy="0 0 0"/>
+        </xacro:inertial_box>
+    </link>
+    <!-- gripper_left -->
+    <joint name="gripper_left_joint" type="revolute">
+        <parent link="slider_left"/>
+        <child link= "gripper_left"/>
+        <origin xyz= "0.2 0 0" rpy= "0 0 0"/>
+        <axis xyz= "0 0 1"/>
+        <limit lower="-1.57" upper="0" effort="10" velocity="0.1"/>
+    </joint>
+    <link name="gripper_left">
+        <visual>
+            <origin xyz= "0.02 0 0.0423" rpy= "0 0 0"/>
+            <geometry>
+                <box size = "0.1 0.025 0.025"/>
+            </geometry>
+            <material name= "cyan"/>
+        </visual>
+        <collision>
+            <origin xyz= "0.02 0 0.0423" rpy= "0 0 0"/>
+            <geometry>
+                <box size = "0.1 0.025 0.025"/>
+            </geometry>
+        </collision>
+        <xacro:inertial_box mass= "0.5" x="0.1" y="0.1" z="0.1">
+            <origin xyz= "0.02 0 0.0423" rpy= "0 0 0"/>
+        </xacro:inertial_box>
+    </link>
+    <!-- gripper_right -->
+    <joint name="gripper_right_joint" type="revolute">
+        <parent link="slider_right"/>
+        <child link= "gripper_right"/>
+        <origin xyz= "0.2 0 0" rpy= "0 0 0"/>
+        <axis xyz= "0 0 1"/>
+        <limit lower="0" upper="1.57" effort="10" velocity="0.1"/>
+    </joint>
+    <link name="gripper_right">
+        <visual>
+            <origin xyz= "0.02 0 0.0423" rpy= "0 0 0"/>
+            <geometry>
+                <box size = "0.1 0.025 0.025"/>
+            </geometry>
+            <material name= "cyan"/>
+        </visual>
+        <collision>
+            <origin xyz= "0.02 0 0.0423" rpy= "0 0 0"/>
+            <geometry>
+                <box size = "0.1 0.025 0.025"/>
+            </geometry>
+        </collision>
+        <xacro:inertial_box mass= "0.5" x="0.1" y="0.1" z="0.1">
+            <origin xyz= "0.02 0 0.0423" rpy= "0 0 0"/>
+        </xacro:inertial_box>
+    </link>
+    <!-- IMU -->
+    <joint name="imu_joint" type="fixed">
+        <parent link="base_link"/>
+        <child link="imu_link"/>
+        <origin xyz="0 0 0.1" rpy="0 0 0"/> <!-- Adjust the position and orientation as needed -->
+    </joint>
+    <link name="imu_link">
+        <visual>
+            <geometry>
+                <box size="0.05 0.05 0.05"/>
+            </geometry>
+            <material name="blue"/>
+        </visual>
+        <collision>
+            <geometry>
+                <box size="0.05 0.05 0.05"/>
+            </geometry>
+        </collision>
+        <inertial>
+            <mass value="0.1"/> <!-- Adjust the mass as needed -->
+            <origin xyz="0 0 0" rpy="0 0 0"/>
+            <inertia ixx="0.0001" ixy="0.0" ixz="0.0" iyy="0.0001" iyz="0.0" izz="0.0001"/> <!-- Adjust the inertia as needed -->
+        </inertial>
+    </link>
 </robot>

File: src/minibot/description/ros2_control.xacro (robot description, xacro)
@@ -11,5 +11,5 @@
                     <param name="baud_rate">57600</param>
                     <param name="timeout_ms">1000</param>
-                    <param name="enc_counts_per_rev">616</param>
+                    <param name="enc_counts_per_rev">3200</param>
             </hardware>
             <joint name="left_wheel_joint">
@@ -25,4 +25,50 @@
                     <param name="min">-10</param>
                     <param name="max">10</param>
+                </command_interface>
+                <state_interface name="position"/>
+                <state_interface name="velocity"/>
+            </joint>
+        </ros2_control>
+        <ros2_control name="GrabberSystem" type="system">
+            <hardware>
+                <plugin>extender_arduino/ExtenderArduinoHardware</plugin>
+                    <param name="joints">slider_left_joint</param>
+                    <param name="platform">platform_joint</param>
+                    <param name="gripper_l">gripper_left_joint</param>
+                    <param name="gripper_r">gripper_right_joint</param>
+                    <param name="loop_rate">30</param>
+                    <param name="device">/dev/ttyACM1</param>
+                    <param name="baud_rate">57600</param>
+                    <param name="timeout_ms">1000</param>
+                    <param name="enc_counts_per_rev">3200</param>
+            </hardware>
+            <joint name="slider_left_joint">
+                <command_interface name="velocity">
+                    <param name="min">-10</param>
+                    <param name="max">10</param>
+                </command_interface>
+                <state_interface name="position"/>
+                <state_interface name="velocity"/>
+            </joint>
+            <!-- <joint name="platform_joint">
+                <command_interface name="velocity">
+                    <param name="min">-10</param>
+                    <param name="max">10</param>
+                </command_interface>
+                <state_interface name="position"/>
+                <state_interface name="velocity"/>
+            </joint> -->
+            <joint name="gripper_left_joint">
+                <command_interface name="position">
+                    <param name="min">0</param>
+                    <param name="max">1.57</param>
+                </command_interface>
+                <state_interface name="position"/>
+                <state_interface name="velocity"/>
+            </joint>
+            <joint name="gripper_right_joint">
+                <command_interface name="position">
+                    <param name="min">-1.57</param>
+                    <param name="max">0</param>
                 </command_interface>
                 <state_interface name="position"/>
