Commit message: updated pid in ros2_control

File: install/minibot/share/minibot/description/camera.xacro (robot description, xacro)
@@ -1 +1,70 @@
-/home/olympusolutions/senior_ws/src/minibot/description/camera.xacro
+<?xml version="1.0"?>
+<robot xmlns:xacro="http://www.ros.org/wiki/xacro" name="robot">
+    <xacro:property name="camera_length"             value="0.01"/>
+    <xacro:property name="camera_width"              value="0.03"/>
+    <xacro:property name="camera_height"             value="0.03"/>
+    <xacro:property name="camera_offset_x"           value="0.5"/>
+    <xacro:property name="camera_offset_z"           value="1.0"/>
+    <!-- Camera -->
+    <joint name="camera_joint" type="fixed">
+        <parent link="chasis"/>
+        <child link="camera_link"/>
+        <origin xyz="${camera_offset_x} 0.0 ${camera_offset_z}" rpy="0 ${pi/4} 0"/>
+    </joint>
+    <link name="camera_link">
+        <visual>
+            <geometry>
+                <box size="${camera_length} ${camera_width} ${camera_height}" />
+            </geometry>
+            <material name="orange"/>
+        </visual>
+    </link>
+    <joint name="camera_optical_joint" type="fixed">
+        <parent link="camera_link"/>
+        <child link="camera_link_optical"/>
+        <origin xyz="0.0 0.0 0.0" rpy="${-pi/2} 0 ${-pi/2}"/>
+    </joint>
+    <link name="camera_link_optical"></link>
+    <!-- Camera in gazebo-->
+    <gazebo reference="camera_link">
+        <sensor name="camera" type="camera">
+            <gz_frame_id>camera_link_optical</gz_frame_id>
+            <pose>0 0 0 0 0 0</pose>
+            <topic>camera/image_raw</topic>
+            <update_rate>30</update_rate>
+            <always_on>1</always_on>
+            <visualize>true</visualize>
+            <camera>
+                <horizontal_fov>1.089</horizontal_fov>
+                <image>
+                    <format>R8G8B8</format>
+                    <width>640</width>
+                    <height>480</height>
+                </image>
+                <clip>
+                    <near>0.05</near>
+                    <far>8.0</far>
+                </clip>
+                <!-- <distortion>
+                    <k1>1.578758331993112829e-01</k1>
+                    <k2>-5.784303605943902360e-01</k2>
+                    <k3>-8.740723680089258069e-03</k3>
+                    <p1>1.359451618091441112e-03</p1>
+                    <p2>1.640043376158566713e-01</p2>
+                    <center>0.5 0.5</center>
+                </distortion>
+                <lens>
+                    <type>pinhole</type>
+                    <scale_to_hfov>false</scale_to_hfov>
+                    <intrinsics>
+                    <fx>4.970870507466349295e+02</fx>
+                    <fy>4.976011127668800782e+02</fy>
+                    <cx>3.168387473166100108e+02</cx>
+                    <cy>2.342740555042151982e+02</cy>
+                    <s>0.0</s>
+                    </intrinsics>
+                </lens> -->
+            </camera>
+        </sensor>
+    </gazebo>
+</robot>

File: install/minibot/share/minibot/description/lidar.xacro (robot description, xacro)
@@ -1 +1,71 @@
-/home/olympusolutions/senior_ws/src/minibot/description/lidar.xacro
+<?xml version="1.0"?>
+<robot xmlns:xacro="http://www.ros.org/wiki/xacro" name="robot">
+    <xacro:property name="lidar_radius"             value="0.025"/>
+    <xacro:property name="lidar_thickness"          value="0.040"/>
+    <xacro:property name="lidar_offset_x"           value="0.230"/>
+    <!-- <xacro:property name="lidar_offset_z"           value="0.098"/> -->
+    <xacro:property name="lidar_offset_z"           value="0.34"/>
+    <!-- Lidar -->
+    <joint name="lidar_joint" type="fixed">
+        <parent link="chasis"/>
+        <child link="lidar_frame"/>
+        <origin xyz="${lidar_offset_x} 0.0 ${lidar_offset_z}" rpy="0 0 ${pi}"/>
+    </joint>
+    <link name="lidar_frame">
+        <visual>
+            <geometry>
+                <cylinder radius="${lidar_radius}" length="${lidar_thickness}"/>
+            </geometry>
+            <material name="orange"/>
+        </visual>
+        <collision>
+            <geometry>
+                <cylinder radius="${lidar_radius}" length="${lidar_thickness}"/>
+            </geometry>
+        </collision>
+        <xacro:inertial_cylinder mass="0.1" radius="${lidar_radius}" length="${lidar_thickness}">
+            <origin xyz="0 0 0" rpy="0 0 0"/>
+        </xacro:inertial_cylinder>
+    </link>
+    <!-- Lidar in gazebo-->
+    <gazebo reference="lidar_frame">
+        <sensor name="lidar" type="gpu_lidar">
+            <gz_frame_id>lidar_frame</gz_frame_id>
+            <pose>0 0 0 0 0 0</pose>
+            <topic>scan</topic>
+            <update_rate>10</update_rate>
+            <always_on>1</always_on>
+            <visualize>true</visualize>
+            <lidar>
+                <scan>
+                    <horizontal>
+                        <samples>360</samples>
+                        <resolution>1</resolution>
+                        <min_angle>-3.14159</min_angle>
+                        <max_angle>3.14159</max_angle>
+                    </horizontal>
+                    <vertical>
+                        <samples>1</samples>
+                        <resolution>0.1</resolution>
+                        <min_angle>0.</min_angle>
+                        <max_angle>0.</max_angle>
+                    </vertical>
+                </scan>
+                <range>
+                    <min>0.08</min>
+                    <max>10.0</max>
+                    <resolution>0.01</resolution>
+                </range>
+                <noise>
+                    <type>gaussian</type>
+                    <mean>0.0</mean>
+                    <stddev>0.01</stddev>
+                </noise>
+            </lidar>
+        <plugin filename="gz-sim-sensors-system"
+                name="gz::sim::systems::Sensors">
+                <render_engine>ogre2</render_engine>
+        </plugin>
+        </sensor>
+    </gazebo>
+</robot>

File: install/minibot/share/minibot/description/robot.urdf.xacro (robot description, xacro)
@@ -1 +1,18 @@
-/home/olympusolutions/senior_ws/src/minibot/description/robot.urdf.xacro
+<?xml version="1.0"?>
+<robot xmlns:xacro="http://www.ros.org/wiki/xacro"  name="robot">
+    <xacro:arg name="use_ros2_control"              default="true"/>
+    <xacro:arg name="use_ros2_control_gz_sim"       default="false"/>
+    <!-- Robot_frames -->
+    <xacro:include filename = "robot_main.xacro" />
+    <!-- Controls -->
+    <xacro:if value="$(arg use_ros2_control)">
+        <xacro:include filename = "ros2_control.xacro" />
+    </xacro:if>
+    <xacro:unless value="$(arg use_ros2_control)">
+        <xacro:include filename = "gz_diff_drive_control.xacro" />
+    </xacro:unless>
+    <!-- Sensors -->
+    <xacro:include filename = "lidar.xacro" />
+    <xacro:include filename = "camera.xacro" />
+    <!-- <xacro:include filename = "depth_camera.xacro" /> -->
+</robot>

File: install/minibot/share/minibot/description/ros2_control.xacro (robot description, xacro)
@@ -1 +1,110 @@
-/home/olympusolutions/senior_ws/src/minibot/description/ros2_control.xacro
+<?xml version="1.0"?>
+<robot xmlns:xacro="http://www.ros.org/wiki/xacro">
+    <xacro:unless value="$(arg use_ros2_control_gz_sim)">
+        <ros2_control name="RobotSystem" type="system">
+            <hardware>
+                <plugin>diffdrive_arduino/DiffDriveArduinoHardware</plugin>
+                    <param name="left_wheel_name">left_wheel_joint</param>
+                    <param name="right_wheel_name">right_wheel_joint</param>
+                    <param name="loop_rate">30</param>
+                    <param name="device">/dev/ttyACM0</param>
+                    <param name="baud_rate">57600</param>
+                    <param name="timeout_ms">1000</param>
+                    <param name="enc_counts_per_rev">3200</param>
+            </hardware>
+            <joint name="left_wheel_joint">
+                <command_interface name="velocity">
+                    <param name="min">-10</param>
+                    <param name="max">10</param>
+                </command_interface>
+                <state_interface name="position"/>
+                <state_interface name="velocity"/>
+            </joint>
+            <joint name="right_wheel_joint">
+                <command_interface name="velocity">
+                    <param name="min">-10</param>
+                    <param name="max">10</param>
+                </command_interface>
+                <state_interface name="position"/>
+                <state_interface name="velocity"/>
+            </joint>
+        </ros2_control>
+        <ros2_control name="GrabberSystem" type="system">
+            <hardware>
+                <plugin>extender_arduino/ExtenderArduinoHardware</plugin>
+                    <param name="joints">slider_left_joint</param>
+                    <param name="platform">platform_joint</param>
+                    <param name="gripper_l">gripper_left_joint</param>
+                    <param name="gripper_r">gripper_right_joint</param>
+                    <param name="loop_rate">30</param>
+                    <param name="device">/dev/ttyACM1</param>
+                    <param name="baud_rate">57600</param>
+                    <param name="timeout_ms">1000</param>
+                    <param name="enc_counts_per_rev">2206</param>
+            </hardware>
+            <joint name="slider_left_joint">
+                <command_interface name="velocity">
+                    <param name="min">-10</param>
+                    <param name="max">10</param>
+                </command_interface>
+                <state_interface name="position"/>
+                <state_interface name="velocity"/>
+            </joint>
+            <!-- <joint name="platform_joint">
+                <command_interface name="velocity">
+                    <param name="min">-10</param>
+                    <param name="max">10</param>
+                </command_interface>
+                <state_interface name="position"/>
+                <state_interface name="velocity"/>
+            </joint> -->
+            <joint name="gripper_left_joint">
+                <command_interface name="position">
+                    <param name="min">0</param>
+                    <param name="max">1.57</param>
+                </command_interface>
+                <state_interface name="position"/>
+                <state_interface name="velocity"/>
+            </joint>
+            <joint name="gripper_right_joint">
+                <command_interface name="position">
+                    <param name="min">-1.57</param>
+                    <param name="max">0</param>
+                </command_interface>
+                <state_interface name="position"/>
+                <state_interface name="velocity"/>
+            </joint>
+        </ros2_control>
+    </xacro:unless>
+    <xacro:if value="$(arg use_ros2_control_gz_sim)">
+        <ros2_control name="minibot_ros2_control" type="system">
+            <hardware>
+                <plugin>gz_ros2_control/GazeboSimSystem</plugin>
+            </hardware>
+            <joint name="left_wheel_joint">
+                <command_interface name="velocity">
+                    <param name="min">-10</param>
+                    <param name="max">10</param>
+                </command_interface>
+                <state_interface name="velocity"/>
+                <state_interface name="position"/>
+            </joint>
+            <joint name="right_wheel_joint">
+                <command_interface name="velocity">
+                    <param name="min">-10</param>
+                    <param name="max">10</param>
+                </command_interface>
+                <state_interface name="velocity"/>
+                <state_interface name="position"/>
+            </joint>
+        </ros2_control>
+        <gazebo>
+            <plugin filename="gz_ros2_control-system"
+                name="gz_ros2_control::GazeboSimROS2ControlPlugin">
+                <parameters>
+                    $(find minibot)/config/controller_gz_sim.yaml
+                </parameters>
+            </plugin>
+        </gazebo>
+    </xacro:if>
+</robot>

File: src/minibot/description/ros2_control.xacro (robot description, xacro)
@@ -7,9 +7,9 @@
                     <param name="left_wheel_name">left_wheel_joint</param>
                     <param name="right_wheel_name">right_wheel_joint</param>
-                    <param name="loop_rate">30</param>
+                    <param name="loop_rate">70</param>
                     <param name="device">/dev/ttyACM0</param>
                     <param name="baud_rate">57600</param>
                     <param name="timeout_ms">1000</param>
-                    <param name="enc_counts_per_rev">3200</param>
+                    <param name="enc_counts_per_rev">7000</param>
             </hardware>
             <joint name="left_wheel_joint">
